File: cad_files/mm2a.sch (KiCad schematic (older format))
At the start: 24 parts, among them J1 DUAL_SWITCH_INV, J1 RELAY, J2 RELAY, J2a SPST, J2b SPST, K1 SPST, K2 DUAL_SWITCH_INV, K3 PushButton

Commit message: #171124
Parts:
- B1: value 750mA -> 800 mA T
- renumbered Cs2 to Cs2a, Cs3 to Cs2b
Changed lines of the file:
@@
 Sheet 1 1
 Title "MM2A gombatermeszto automatika"
-Date "14 sep 2017"
+Date "24 nov 2017"
 Rev "1.0"
 Comp "Pozsár Zsolt"
@@
 P 8650 2000
 F 0 "B1" V 8750 2100 50  0000 C CNN
-F 1 "750mA" V 8550 2000 50  0000 C CNN
+F 1 "800 mA T" V 8550 2000 50  0000 C CNN
 F 2 "" H 8650 2000 60  0000 C CNN
 F 3 "" H 8650 2000 60  0000 C CNN
@@
 $EndComp
 $Comp
-L CONN_3 Cs2
+L CONN_3 Cs2a
 U 1 1 59BAC0FF
 P 1000 2200
-F 0 "Cs2" H 950 1950 50  0000 C CNN
+F 0 "Cs2a" H 950 1950 50  0000 C CNN
 F 1 "CONN_3" V 1050 2200 40  0001 C CNN
 F 2 "" H 1000 2200 60  0000 C CNN
@@
 $EndComp
 $Comp
-L CONN_2 Cs3
+L CONN_2 Cs2b
 U 1 1 59BAC12C
 P 9450 1150
-F 0 "Cs3" V 9350 1400 40  0000 C CNN
+F 0 "Cs2b" V 9350 1400 40  0000 C CNN
 F 1 "CONN_2" V 9500 1150 40  0001 C CNN
 F 2 "" H 9450 1150 60  0000 C CNN

Commit message: #171210
Parts:
- removed Cs2a: CONN_3, symbol CONN_3
- removed Cs2b: CONN_2, symbol CONN_2
- removed IK1: SPST, ~, symbol SPST
- added Cs2: CONN_6, symbol CONN_6
- added K4: TSGM1, ~, symbol TIMER
- J1, J2: value RELAY -> Finder 40.52
- La1: value GLIMM -> TN-0,3
Connections:
- net labels added: GND
- net labels removed: HT
- wire segments 67 -> 92
Other:
- note removed: "Időkapcsoló tápfeszültség\n230V AC"
- moved on the sheet: C1, Cs1, D1, D2, D3, D4, D5, J1, J1A, J1B, J2, J2a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

Commit message: 
Parts:
- removed C1: 4700u 25V, ~, symbol CAPAPOL
- removed Cs1: CONN_2, symbol CONN_2
- removed Cs2: CONN_6, symbol CONN_6
- removed La1: TN-0,3, glimm, symbol GLIMM
- removed La2: 26V 120mA, lamp, symbol LAMP
- added C?: CP, symbol CP
- added J?: Screw_Terminal_01x06, symbol Screw_Terminal_01x06
- added J?: Screw_Terminal_01x02, symbol Screw_Terminal_01x02
- added LA?: Lamp, symbol Lamp
- added La?: glimm, glimm, symbol glimm
- B1: symbol FUSE-EU -> Fuse-EU
- R1: symbol R -> R-RESCUE-mm2a
Connections:
- net labels added: GNDD
- net labels removed: GND
- wire segments 92 -> 86
Other:
- moved on the sheet: D1, D2, D3, D4, D5, J1, J1A, J1B, J2, J2a, J2b, K1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

Commit message: #180318
Parts:
- removed D1, D2: 1N4001, ~, symbol DIODE
- removed D3, D4, D5: D237, ~, symbol DIODE
- added D1, D2, D6: 1N4001, symbol D
- added D3, D4, D5: D237, symbol D
- C1: renamed from C?; value CP -> 4700u 40V
- La2: renamed from LA?; value Lamp -> 24V 0,1A
- gave numbers to parts that had none: 3
- renumbered J2a to J2A, J2b to J2B, K4 to U1
Connections:
- wire segments 86 -> 74
Other:
- note added: "Belső\n\n\nKülső"
- note added: "Vezérlés"
- note removed: "Vezérlés\n\nBelső\nKülső"
- moved on the sheet: B1, J1B, J2A, J2B, K3, La1, La2, R1, Tr1, Tr2

Commit message: #180515
Parts:
- removed C1: 4700u 40V, symbol CP
- removed Cs1: Screw_Terminal_01x06, symbol Screw_Terminal_01x06
- removed Cs2: Screw_Terminal_01x02, symbol Screw_Terminal_01x02
- removed D1, D2, D6: 1N4001, symbol D
- removed D3, D4, D5: D237, symbol D
- removed J1, K2: DUAL_SWITCH_INV, ~, symbol DUAL_SWITCH_INV
- removed unit 2 of J1
- removed La1: glimm, glimm, symbol glimm
- removed La2: 24V 0,1A, symbol Lamp
- added C1, C2: 4700u 25V, ~, symbol CAPAPOL
- added Cs1: CONN_2, symbol CONN_2
- added Cs2: CONN_6, symbol CONN_6
- added D1, D2, D6: 1N4001, ~, symbol DIODE
- added D3, D4, D5: D237, ~, symbol DIODE
- added J1a, J1b, K2a, K2b: SWITCH_INV, ~, symbol SWITCH_INV
- added K1b: SPST, ~, symbol SPST
- added La1: TN-0,3, glimm, symbol GLIMM
- added La2: 26V 120mA, lamp, symbol LAMP
- B1: symbol Fuse-EU -> FUSE-EU
- R1: symbol R-RESCUE-mm2a -> R
- renumbered J2A to J2a, J2B to J2b, K1 to K1a, U1 to K4
Connections:
- net labels added: GND
- net labels removed: GNDD
- wire segments 74 -> 101
Other:
- note added: "+12V"
- note added: "230V AC"
- note added: "Belső\nKülső"
- note removed: "Belső\n\n\nKülső"
- moved on the sheet: J1, J2, J2a, J2b, K1a, K3, K4, R1, Tr1, Tr2

Commit message: #181222
Parts:
- removed C1, C2: 4700u 25V, ~, symbol CAPAPOL
- added C1, C2: 4700u, symbol CP
- B1: symbol FUSE-EU -> Fuse-EU
- La1: symbol GLIMM -> glimm
- La2: symbol LAMP -> Lamp
- R1: symbol R -> R-RESCUE-mm2a
Connections:
- net labels added: GNDD
- net labels removed: GND
- wire segments 101 -> 79
Other:
- note added: "Belső\n |\nKülső"
- note removed: "Belső\nKülső"
